File: keyboard.kicad_sch (KiCad schematic)
At the start: 176 parts, among them J1 USB_C_Receptacle_USB2.0_16P, J2 Conn_01x04, J3 Conn_01x05, U1 XC6206PxxxMR, U2 SRV05-4, U3 RP2040, U4 W25Q128JVS, Y1 Crystal_GND24

Commit message: changes to schematics
Parts:
- removed S1: MX_stab, PCM_marbastlib-mx:STAB_MX_P_1.5u, symbol PCM_marbastlib-mx:MX_stab
- removed S2, S3: MX_stab, PCM_marbastlib-mx:STAB_MX_P_1.75u, symbol PCM_marbastlib-mx:MX_stab
- removed S4, S5: MX_stab, PCM_marbastlib-mx:STAB_MX_P_2u, symbol PCM_marbastlib-mx:MX_stab
Other:
- note added: "stabilizer for keys (1.5 u)"
- title: (none) -> Custom Keyboard for my macbook
